File: Main_board/Main_board.sch (KiCad schematic (older format))
At the start: 65 parts, among them J1 USB_B_Micro, Q1 Q_PMOS_GDS, Q2 Q_NMOS_GDS, U1 ATmega328-AU, U2 FT232RL, U3 XR2206, U4 TXS0104, U5 MX25L51245G, U6 74LS125, Y1 20Mhz

Commit message: ENH: Component placed
Parts:
- C11, C12: footprint Capacitor_SMD:C_1206_3216Metric -> Capacitor_SMD:C_0603_1608Metric
- C6: value 10n -> 10u; footprint Capacitor_SMD:C_1206_3216Metric -> Capacitor_SMD:CP_Elec_4x5.4
- C9: footprint Capacitor_SMD:CP_Elec_4x5.4 -> Capacitor_SMD:C_0603_1608Metric
Connections:
- net 12v_on: now also U1.2 (PD4); no longer U1.11 (PD7)
- net btn1: now also U1.12 (PB0); no longer U1.25 (PC2)
- net btn2: now also U1.13 (PB1); no longer U1.26 (PC3)
- net hall: now also U1.25 (PC2); no longer U1.12 (PB0)
- net led1: now also U1.9 (PD5); no longer U1.2 (PD4)
- net led2: now also U1.10 (PD6); no longer U1.9 (PD5)
- net led3: now also U1.11 (PD7); no longer U1.10 (PD6)
- net seq: now also U1.26 (PC3); no longer U1.13 (PB1)
Changed lines of the file:
@@
 	13250 6700 15400 6700
 Text Label 9300 1700 0    50   ~ 0
-hall
+btn1
 Text Label 9300 1800 0    50   ~ 0
-seq
+btn2
 Text Label 9300 1900 0    50   ~ 0
 uart_on
@@
 press
 Text Label 9300 2800 0    50   ~ 0
-btn1
+hall
 Text Label 9300 2900 0    50   ~ 0
-btn2
+seq
 Text Label 9300 3000 0    50   ~ 0
 sda
@@
 pneuma
 Text Label 9300 3800 0    50   ~ 0
+12v_on
+Text Label 9300 3900 0    50   ~ 0
 led1
-Text Label 9300 3900 0    50   ~ 0
+Text Label 9300 4000 0    50   ~ 0
 led2
-Text Label 9300 4000 0    50   ~ 0
-led3
 Wire Wire Line
 	7650 1350 8000 1350
@@
 	13700 7800 13700 7750
 Text Label 9300 4100 0    50   ~ 0
-12v_on
+led3
 Wire Wire Line
 	9300 4100 9250 4100
@@
 F 0 "C11" H 3465 6146 50  0000 L CNN
 F 1 "10n" H 3465 6055 50  0000 L CNN
-F 2 "Capacitor_SMD:C_1206_3216Metric" H 3388 5950 50  0001 C CNN
+F 2 "Capacitor_SMD:C_0603_1608Metric" H 3388 5950 50  0001 C CNN
 F 3 "~" H 3350 6100 50  0001 C CNN
 	1    3350 6100
@@
 F 0 "C12" H 4915 6146 50  0000 L CNN
 F 1 "10n" H 4915 6055 50  0000 L CNN
-F 2 "Capacitor_SMD:C_1206_3216Metric" H 4838 5950 50  0001 C CNN
+F 2 "Capacitor_SMD:C_0603_1608Metric" H 4838 5950 50  0001 C CNN
 F 3 "~" H 4800 6100 50  0001 C CNN
 	1    4800 6100
@@
 F 0 "C9" H 2115 3246 50  0000 L CNN
 F 1 "4.7n" H 2115 3155 50  0000 L CNN
-F 2 "Capacitor_SMD:CP_Elec_4x5.4" H 2038 3050 50  0001 C CNN
+F 2 "Capacitor_SMD:C_0603_1608Metric" H 2038 3050 50  0001 C CNN
 F 3 "~" H 2000 3200 50  0001 C CNN
 	1    2000 3200
@@
 P 2850 2150
 F 0 "C6" V 3105 2150 50  0000 C CNN
-F 1 "10n" V 3014 2150 50  0000 C CNN
-F 2 "Capacitor_SMD:C_1206_3216Metric" H 2888 2000 50  0001 C CNN
+F 1 "10u" V 3014 2150 50  0000 C CNN
+F 2 "Capacitor_SMD:CP_Elec_4x5.4" H 2888 2000 50  0001 C CNN
 F 3 "~" H 2850 2150 50  0001 C CNN
 	1    2850 2150

Commit message: WIP: still routing
Connections:
- net press is gone; now on net pressure: U1.23 (PC0)
Changed lines of the file:
@@
 xtal2
 Text Label 9300 2600 0    50   ~ 0
-press
+pressure
 Text Label 9300 2800 0    50   ~ 0
 hall
