File: Main_board/Main_board.kicad_pcb (KiCad board)
At the start: 2 copper layers, 59.9 x 94.1 mm, 65 parts, among them J1 USB_B_Micro, Q1 Q_PMOS_GDS, Q2 Q_NMOS_GDS, U1 ATmega328-AU, U2 FT232RL, U3 XR2206, U4 TXS0104, U5 MX25L51245G, U6 74LS125, Y1 20Mhz

Commit message: WIP: routing
Parts:
- turned C11 to 180 degrees
- turned C12 to 180 degrees
Routing:
- net /rx_periph: track 0.00 -> 42.5 mm
- net +5V: track 0.00 -> 21.9 mm
- net /scl: track 0.00 -> 19.4 mm, vias 0 -> 1
- net /sda: track 0.00 -> 16.6 mm, vias 0 -> 1
- net /xtal2: track 0.00 -> 16.1 mm
- net /btn2: track 0.00 -> 15.3 mm
- net /btn1: track 0.00 -> 13.7 mm
- net Net-(RV3-Pad1): track 0.00 -> 12.7 mm
- net Net-(C10-Pad1): track 0.00 -> 12.4 mm
- net /xtal1: track 0.00 -> 11.8 mm
- net Net-(R7-Pad1): track 0.00 -> 8.50 mm
- net Net-(R8-Pad2): track 0.00 -> 8.16 mm
- net /uart_off: track 0.00 -> 6.45 mm
- net Net-(RV2-Pad1): track 0.00 -> 5.90 mm
- net /led3: track 0.00 -> 5.41 mm
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
Commit message: WIP: still routing
Parts:
- moved Q1 29.2 mm to (157.0, 109.1)
Connections:
- U1 pad 23: /press -> /pressure
Routing:
- net +5V: track 21.9 -> 181.4 mm, vias 0 -> 6
- net +12V: track 0.00 -> 83.1 mm, vias 0 -> 2
- net /uart_on: track 0.00 -> 74.9 mm, vias 0 -> 4
- net /rx_mcu: track 4.04 -> 78.7 mm, vias 0 -> 2
- net /tx_mcu: track 0.00 -> 67.8 mm, vias 0 -> 2
- net /12v_on: track 0.00 -> 60.5 mm
- net /hall: track 0.00 -> 60.1 mm, vias 0 -> 3
- net /pneuma: track 0.00 -> 59.1 mm, vias 0 -> 2
- net /bat_volt: track 0.00 -> 57.2 mm, vias 0 -> 2
- net /despin: track 0.00 -> 56.6 mm, vias 0 -> 3
- net +3V3: track 0.00 -> 53.1 mm
- net Net-(TELEM1-Pad2): track 0.00 -> 49.6 mm
- net /bat_current: track 0.00 -> 47.2 mm, vias 0 -> 2
- net Net-(J1-Pad3): track 0.00 -> 33.0 mm, vias 0 -> 2
- net /sck: track 0.00 -> 31.8 mm, vias 0 -> 2
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
Commit message: ENH: finished routing
Parts:
- added REF**: MountingHole_2.2mm_M2, MountingHole:MountingHole_2.2mm_M2, F.Cu at (126.0, 54.6)
- added REF**: MountingHole_2.2mm_M2, MountingHole:MountingHole_2.2mm_M2, F.Cu at (180.8, 54.6)
- added REF**: MountingHole_2.2mm_M2, MountingHole:MountingHole_2.2mm_M2, F.Cu at (126.0, 143.7)
- added REF**: MountingHole_2.2mm_M2, MountingHole:MountingHole_2.2mm_M2, F.Cu at (180.8, 143.7)
- renumbered ALIM1 to ALIM, GPS1 to GPS, ICSP1 to ICSP, IMU1 to IMU, PRESS1 to PRESS, SCREEN1 to SCREEN, SEQ1 to SEQ, TELEM1 to TELEM, TO_AN_BOARD1 to TO_AN_BOARD
Routing:
- net /tx_usb: track 0.00 -> 111.9 mm, vias 0 -> 2
- net /rx_usb: track 2.25 -> 101.2 mm, vias 0 -> 2
- net +5V: track 181.4 -> 246.4 mm, vias 6 -> 9
- net /reset: track 16.3 -> 43.9 mm, vias 2 -> 6
- net /miso: track 22.7 -> 44.0 mm, vias 2 -> 3
- net /mosi: track 28.1 -> 46.9 mm, vias 1 -> 2
- net GND: track 0.00 -> 18.2 mm, vias 0 -> 11
- net /sck: track 31.8 -> 50.0 mm, vias 2 -> 3
- net (no net): track 0.00 -> 3.84 mm
- net /rx_mcu: track 78.7 -> 80.3 mm
- net Net-(D3-Pad1): track 23.6 -> 24.3 mm
- net Net-(D4-Pad1): track 17.0 -> 17.6 mm
- added copper zone on B.Cu, net GND
- added copper zone on F.Cu, net GND
Other:
- board text added: "AERIS III"
- board text added: "Main board"
