File: Sequencer_board/Sequencer_board.sch (KiCad schematic (older format))
At the start: 27 parts

Commit message: ENH: AN board finished
Parts:
- removed J? (x2): Conn_01x02_Male, symbol Connector:Conn_01x02_Male
- added C4: 100n, Capacitor_SMD:C_0603_1608Metric, symbol Device:C
- added HALL1: Conn_01x03, Connector_PinHeader_2.54mm:PinHeader_1x03_P2.54mm_Vertical, symbol Connector_Generic:Conn_01x03
- added J1, J3: Conn_01x02, Connector_PinHeader_2.54mm:PinHeader_1x02_P2.54mm_Vertical, symbol Connector_Generic:Conn_01x02
- added J2: Conn_01x06, Connector_PinHeader_2.54mm:PinHeader_1x06_P2.54mm_Vertical, symbol Connector_Generic:Conn_01x06
- added Q7: Q_NMOS_GDS, Package_TO_SOT_SMD:TO-252-2, symbol Device:Q_NMOS_GDS
- added R8, R9: 10k, Resistor_SMD:R_0603_1608Metric, symbol Device:R
- C1, C2, C3: renamed from C?; value CP -> 470u; footprint (none) -> Capacitor_THT:CP_Radial_D10.0mm_P5.00mm
- Q1, Q2, Q3, Q4, Q5, Q6: renamed from Q?; footprint (none) -> Package_TO_SOT_SMD:TO-252-2
- R1: renamed from R?; value R -> 10k; footprint (none) -> Resistor_SMD:R_0603_1608Metric
- R2: renamed from R?; value R -> 56k; footprint (none) -> Resistor_THT:R_Axial_DIN0207_L6.3mm_D2.5mm_P2.54mm_Vertical
- R3, R5, R7: renamed from R?; value R -> 100k; footprint (none) -> Resistor_SMD:R_0603_1608Metric
- R4: renamed from R?; value R -> 33k; footprint (none) -> Resistor_THT:R_Axial_DIN0207_L6.3mm_D2.5mm_P2.54mm_Vertical
- R6: renamed from R?; value R -> 18k; footprint (none) -> Resistor_THT:R_Axial_DIN0207_L6.3mm_D2.5mm_P2.54mm_Vertical
- RV1, RV2, RV3: renamed from RV?; value R_POT_TRIM -> 10k; footprint (none) -> Potentiometer_THT:Potentiometer_Bourns_3296W_Vertical
- U1: renamed from U?; footprint (none) -> Package_SO:SOIC-14_3.9x8.7mm_P1.27mm
- U2: renamed from U?; footprint (none) -> Package_SO:SSOP-8_2.95x2.8mm_P0.65mm
Connections:
- net VCC is gone; now on net +5V: U2.8 (VCC), U2.8 (VCC)
- net +5V: now also U1.4 (V+), C4.1, HALL1.3 (Pin_3), J2.2 (Pin_2), R8.1, R9.1
- net AN_shutdown: now also U2.1, U2.5; no longer U2.1, U2.5
- net GND: now also U1.11 (V-), C4.2, HALL1.1 (Pin_1), J2.6 (Pin_6), Q7.3 (S)
- net hall: now also J2.3 (Pin_3), Q7.2 (D), R9.2
- net pneuma: now also U2.3, J2.4 (Pin_4); no longer Q3.1 (G), U2.3, U2.7
- net at R7.1, U1.7: now also U2.6; no longer U2.2
- net at R5.1, U1.8: now also U2.2; no longer U2.6
- net at Q3.2 (D): now also J1.2 (Pin_2)
- net at Q5.2 (D): now also J3.2 (Pin_2)
- new net: HALL1.2 (Pin_2), Q7.1 (G), R8.2
- new net +24V: J1.1 (Pin_1), J2.1 (Pin_1), J3.1 (Pin_1)
- new net despin: J2.5 (Pin_5), Q3.1 (G), U2.7
Other:
- moved on the sheet: C1, C2, C3, Q1, Q2, Q3, Q4, Q5, Q6, R1, R2, R3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
